File: board/SSR8A.sch (KiCad schematic (older format))
At the start: 4 parts, among them U1 PCF8574

Commit message: WIP
Parts:
- added C5: 100n, Capacitors_SMD:C_0805, symbol C
- added D1: LED, LEDs:LED_0805, symbol LED
- added R1: 270R, Resistors_SMD:R_0805, symbol R
- added X1: I2C, device.farm:Micro-Match-FOB-4, symbol I2C
- IN1: footprint device.farm:DG301-5.0-02 -> device.farm:DG142R-2-5.08
- renumbered R1 to R2, R2 to R3
Connections:
- net ESP/GPIO4: now also R1.2
- net GND: now also C5.2, D1.1 (K), X1.1 (GND)
- net SCL: now also X1.2 (SCL)
- net SDA: now also X1.3 (SDA)
- net 3V3 renamed VCC
- net VCC: now also C5.1, X1.4 (3V3)
- new net: D1.2 (A), R1.1
- no-connect marks 6 -> 5
Other:
- moved on the sheet: R2, R3
