File: board/esp-mains.sch (KiCad schematic (older format))
At the start: 26 parts, among them P1 USB_OTG, Q1 MMBT3904, Q2 MMBT3904, U2 RT9193, U3 HLK-PM01, U4 ESP-12, U5 CH340G, X1 12MHz

Commit message: WIP
Parts:
- added C8, C9: 47u, Capacitors_SMD:C_0805, symbol C
- renumbered Q1 to Q2, Q2 to Q3, U2 to U1, U3 to U2
Connections:
- net GND: now also C8.2, C9.2
- net VCC: now also C8.1, C9.1
Changed lines of the file:
@@
 EESchema Schematic File Version 2
+LIBS:CR1TS1A-rescue
 LIBS:power
 LIBS:device
@@
 LIBS:valves
 LIBS:device.farm
-LIBS:SSR8A-cache
+LIBS:CR1TS1A-cache
 EELAYER 25 0
 EELAYER END
 $Descr A4 11693 8268
 encoding utf-8
-Sheet 2 10
+Sheet 2 2
 Title ""
 Date ""
@@
 $EndComp
 $Comp
-L HLK-PM01 U3
+L HLK-PM01 U2
 U 1 1 5777B23B
 P 4050 2200
-F 0 "U3" H 4050 2637 60  0000 C CNN
+F 0 "U2" H 4050 2637 60  0000 C CNN
 F 1 "HLK-PM01" H 4050 2531 60  0000 C CNN
 F 2 "device.farm:HLK-PM01" H 4050 2200 60  0001 C CNN
@@
 $EndComp
 $Comp
-L GND #PWR04
+L GND #PWR12
 U 1 1 5777B23D
 P 4550 2350
-F 0 "#PWR04" H 4550 2100 50  0001 C CNN
+F 0 "#PWR12" H 4550 2100 50  0001 C CNN
 F 1 "GND" V 4555 2222 50  0000 R CNN
 F 2 "" H 4550 2350 50  0000 C CNN
@@
 $EndComp
 $Comp
-L GND #PWR05
+L GND #PWR9
 U 1 1 5777B244
 P 3450 5400
-F 0 "#PWR05" H 3450 5150 50  0001 C CNN
+F 0 "#PWR9" H 3450 5150 50  0001 C CNN
 F 1 "GND" H 3455 5227 50  0000 C CNN
 F 2 "" H 3450 5400 50  0000 C CNN
@@
 $EndComp
 $Comp
-L GND #PWR06
+L GND #PWR10
 U 1 1 5777B245
 P 3900 5400
-F 0 "#PWR06" H 3900 5150 50  0001 C CNN
+F 0 "#PWR10" H 3900 5150 50  0001 C CNN
 F 1 "GND" H 3905 5227 50  0000 C CNN
 F 2 "" H 3900 5400 50  0000 C CNN
@@
 $EndComp
 $Comp
-L RT9193 U2
+L RT9193 U1
 U 1 1 5777B246
 P 3450 4950
-F 0 "U2" H 3450 5387 60  0000 C CNN
+F 0 "U1" H 3450 5387 60  0000 C CNN
 F 1 "RT9193" H 3450 5281 60  0000 C CNN
 F 2 "TO_SOT_Packages_SMD:SOT-23-5" H 3450 4950 60  0001 C CNN
@@
 $EndComp
 $Comp
-L GND #PWR07
+L GND #PWR8
 U 1 1 5777B247
 P 2600 5400
-F 0 "#PWR07" H 2600 5150 50  0001 C CNN
+F 0 "#PWR8" H 2600 5150 50  0001 C CNN
 F 1 "GND" H 2605 5227 50  0000 C CNN
 F 2 "" H 2600 5400 50  0000 C CNN
@@
 $EndComp
 $Comp
-L GND #PWR08
+L GND #PWR11
 U 1 1 5777B249
 P 4300 5400
-F 0 "#PWR08" H 4300 5150 50  0001 C CNN
+F 0 "#PWR11" H 4300 5150 50  0001 C CNN
 F 1 "GND" H 4305 5227 50  0000 C CNN
 F 2 "" H 4300 5400 50  0000 C CNN
@@
 TX
 $Comp
-L GND #PWR09
+L GND #PWR20
 U 1 1 5777B24B
 P 6600 2750
-F 0 "#PWR09" H 6600 2500 50  0001 C CNN
+F 0 "#PWR20" H 6600 2500 50  0001 C CNN
 F 1 "GND" H 6605 2577 50  0000 C CNN
 F 2 "" H 6600 2750 50  0000 C CNN
@@
 $EndComp
 $Comp
-L GND #PWR010
+L GND #PWR5
 U 1 1 5777B24D
 P 1600 3500
-F 0 "#PWR010" H 1600 3250 50  0001 C CNN
+F 0 "#PWR5" H 1600 3250 50  0001 C CNN
 F 1 "GND" H 1605 3327 50  0000 C CNN
 F 2 "" H 1600 3500 50  0000 C CNN
@@
 $EndComp
 $Comp
-L GND #PWR011
+L GND #PWR13
 U 1 1 5777B24F
 P 4900 5400
-F 0 "#PWR011" H 4900 5150 50  0001 C CNN
+F 0 "#PWR13" H 4900 5150 50  0001 C CNN
 F 1 "GND" H 4905 5227 50  0000 C CNN
 F 2 "" H 4900 5400 50  0000 C CNN
@@
 $EndComp
 $Comp
-L MMBT3904 Q1
+L MMBT3904 Q2
 U 1 1 5777B252
 P 9800 2100
-F 0 "Q1" H 10050 2200 50  0000 C CNN
+F 0 "Q2" H 10050 2200 50  0000 C CNN
 F 1 "MMBT3904" H 10200 2100 50  0000 C CNN
 F 2 "TO_SOT_Packages_SMD:SOT-23" H 10500 1450 50  0001 C CIN
@@
 $EndComp
 $Comp
-L MMBT3904 Q2
+L MMBT3904 Q3
 U 1 1 5777B253
 P 9800 2800
-F 0 "Q2" H 10050 2900 50  0000 C CNN
+F 0 "Q3" H 10050 2900 50  0000 C CNN
 F 1 "MMBT3904" H 10200 2800 50  0000 C CNN
 F 2 "TO_SOT_Packages_SMD:SOT-23" H 10500 2150 50  0001 C CIN
@@
 $EndComp
 $Comp
-L GND #PWR012
+L GND #PWR21
 U 1 1 5777B25A
 P 7550 5200
-F 0 "#PWR012" H 7550 4950 50  0001 C CNN
+F 0 "#PWR21" H 7550 4950 50  0001 C CNN
 F 1 "GND" H 7555 5027 50  0000 C CNN
 F 2 "" H 7550 5200 50  0000 C CNN
@@
 $EndComp
 $Comp
-L GND #PWR013
+L GND #PWR24
 U 1 1 5777B260
 P 9700 5500
-F 0 "#PWR013" H 9700 5250 50  0001 C CNN
+F 0 "#PWR24" H 9700 5250 50  0001 C CNN
 F 1 "GND" H 9705 5327 50  0000 C CNN
 F 2 "" H 9700 5500 50  0000 C CNN
@@
 $EndComp
 $Comp
-L GND #PWR014
+L GND #PWR23
 U 1 1 5777B262
 P 9700 5200
-F 0 "#PWR014" H 9700 4950 50  0001 C CNN
+F 0 "#PWR23" H 9700 4950 50  0001 C CNN
 F 1 "GND" H 9705 5027 50  0000 C CNN
 F 2 "" H 9700 5200 50  0000 C CNN
@@
 $EndComp
 $Comp
-L GND #PWR015
+L GND #PWR4
 U 1 1 5777B266
 P 1500 3500
-F 0 "#PWR015" H 1500 3250 50  0001 C CNN
+F 0 "#PWR4" H 1500 3250 50  0001 C CNN
 F 1 "GND" H 1505 3327 50  0000 C CNN
 F 2 "" H 1500 3500 50  0000 C CNN
@@
 $EndComp
 $Comp
-L VCC #PWR016
+L VCC #PWR25
 U 1 1 5777BAC2
 P 9800 4400
-F 0 "#PWR016" H 9800 4250 50  0001 C CNN
+F 0 "#PWR25" H 9800 4250 50  0001 C CNN
 F 1 "VCC" V 9817 4528 50  0000 L CNN
 F 2 "" H 9800 4400 50  0000 C CNN
@@
 $EndComp
 $Comp
-L VCC #PWR017
+L VCC #PWR22
 U 1 1 5777C042
 P 7600 1750
-F 0 "#PWR017" H 7600 1600 50  0001 C CNN
+F 0 "#PWR22" H 7600 1600 50  0001 C CNN
 F 1 "VCC" V 7617 1878 50  0000 L CNN
 F 2 "" H 7600 1750 50  0000 C CNN
@@
 $EndComp
 $Comp
-L VCC #PWR018
+L VCC #PWR19
 U 1 1 5777C582
 P 6600 1750
-F 0 "#PWR018" H 6600 1600 50  0001 C CNN
+F 0 "#PWR19" H 6600 1600 50  0001 C CNN
 F 1 "VCC" V 6618 1877 50  0000 L CNN
 F 2 "" H 6600 1750 50  0000 C CNN
@@
 $EndComp
 $Comp
-L VCC #PWR019
+L VCC #PWR16
 U 1 1 5777C817
-P 6450 5200
-F 0 "#PWR019" H 6450 5050 50  0001 C CNN
-F 1 "VCC" V 6468 5327 50  0000 L CNN
-F 2 "" H 6450 5200 50  0000 C CNN
-F 3 "" H 6450 5200 50  0000 C CNN
-	1    6450 5200
-	0    -1   -1   0
-$EndComp
-$Comp
-L VCC #PWR020
+P 6050 5200
+F 0 "#PWR16" H 6050 5050 50  0001 C CNN
+F 1 "VCC" V 6068 5327 50  0000 L CNN
+F 2 "" H 6050 5200 50  0000 C CNN
+F 3 "" H 6050 5200 50  0000 C CNN
+	1    6050 5200
+	0    -1   -1   0
+$EndComp
+$Comp
+L VCC #PWR14
 U 1 1 5777D0FB
 P 5050 4800
-F 0 "#PWR020" H 5050 4650 50  0001 C CNN
+F 0 "#PWR14" H 5050 4650 50  0001 C CNN
 F 1 "VCC" V 5067 4928 50  0000 L CNN
 F 2 "" H 5050 4800 50  0000 C CNN
@@
 GPIO5
 $Comp
-L GND #PWR021
+L GND #PWR7
 U 1 1 5778ED26
 P 1850 2300
-F 0 "#PWR021" H 1850 2050 50  0001 C CNN
+F 0 "#PWR7" H 1850 2050 50  0001 C CNN
 F 1 "GND" V 1855 2127 50  0000 C CNN
 F 2 "" H 1850 2300 50  0000 C CNN
@@
 $EndComp
 $Comp
-L PWR_FLAG #FLG022
+L PWR_FLAG #FLG2
 U 1 1 5778ED65
 P 1850 2300
-F 0 "#FLG022" H 1850 2395 50  0001 C CNN
+F 0 "#FLG2" H 1850 2395 50  0001 C CNN
 F 1 "PWR_FLAG" V 1850 2650 50  0000 C CNN
 F 2 "" H 1850 2300 50  0000 C CNN
@@
 $EndComp
 $Comp
-L VCC #PWR023
+L VCC #PWR6
 U 1 1 57790C33
 P 1850 2100
-F 0 "#PWR023" H 1850 1950 50  0001 C CNN
+F 0 "#PWR6" H 1850 1950 50  0001 C CNN
 F 1 "VCC" V 1868 2227 50  0000 L CNN
 F 2 "" H 1850 2100 50  0000 C CNN
@@
 $EndComp
 $Comp
-L PWR_FLAG #FLG024
+L PWR_FLAG #FLG1
 U 1 1 57790FA9
 P 1850 2100
-F 0 "#FLG024" H 1850 2195 50  0001 C CNN
+F 0 "#FLG1" H 1850 2195 50  0001 C CNN
 F 1 "PWR_FLAG" V 1850 2450 50  0000 C CNN
 F 2 "" H 1850 2100 50  0000 C CNN
@@
 5V
 $Comp
-L PWR_FLAG #FLG025
+L PWR_FLAG #FLG3
 U 1 1 58F96095
 P 1850 2500
-F 0 "#FLG025" H 1850 2595 50  0001 C CNN
+F 0 "#FLG3" H 1850 2595 50  0001 C CNN
 F 1 "PWR_FLAG" V 1850 2850 50  0000 C CNN
 F 2 "" H 1850 2500 50  0000 C CNN
@@
 $EndComp
 $Comp
-L GND #PWR026
+L GND #PWR18
 U 1 1 58F96138
 P 6400 2550
-F 0 "#PWR026" H 6400 2300 50  0001 C CNN
+F 0 "#PWR18" H 6400 2300 50  0001 C CNN
 F 1 "GND" H 6405 2377 50  0001 C CNN
 F 2 "" H 6400 2550 50  0000 C CNN
@@
 $EndComp
 $Comp
-L GND #PWR027
+L GND #PWR15
 U 1 1 58F96895
 P 5850 2550
-F 0 "#PWR027" H 5850 2300 50  0001 C CNN
+F 0 "#PWR15" H 5850 2300 50  0001 C CNN
 F 1 "GND" H 5855 2377 50  0000 C CNN
 F 2 "" H 5850 2550 50  0000 C CNN
@@
 	5000 4600 5000 4800
 Connection ~ 5000 4800
+$Comp
+L C C9
+U 1 1 5A74BDF9
+P 6350 5400
+F 0 "C9" H 6500 5450 50  0000 L CNN
+F 1 "47u" H 6465 5355 50  0000 L CNN
+F 2 "Capacitors_SMD:C_0805" H 6388 5250 50  0001 C CNN
+F 3 "" H 6350 5400 50  0000 C CNN
+	1    6350 5400
+	1    0    0    -1
+$EndComp
+$Comp
+L C C8
+U 1 1 5A74BEDA
+P 6150 5400
+F 0 "C8" H 5950 5450 50  0000 L CNN
+F 1 "47u" H 5900 5350 50  0000 L CNN
+F 2 "Capacitors_SMD:C_0805" H 6188 5250 50  0001 C CNN
+F 3 "" H 6150 5400 50  0000 C CNN
+	1    6150 5400
+	1    0    0    -1
+$EndComp
+$Comp
+L GND #PWR17
+U 1 1 5A74BFA4
+P 6250 5650
+F 0 "#PWR17" H 6250 5400 50  0001 C CNN
+F 1 "GND" H 6255 5477 50  0000 C CNN
+F 2 "" H 6250 5650 50  0000 C CNN
+F 3 "" H 6250 5650 50  0000 C CNN
+	1    6250 5650
+	1    0    0    -1
+$EndComp
+Wire Wire Line
+	6050 5200 6450 5200
+Wire Wire Line
+	6350 5250 6350 5200
+Connection ~ 6350 5200
+Wire Wire Line
+	6150 5250 6150 5200
+Connection ~ 6150 5200
+Wire Wire Line
+	6250 5650 6250 5550
+Wire Wire Line
+	6150 5550 6350 5550
+Connection ~ 6250 5550
 $EndSCHEMATC

Commit message: WIP
Parts:
- removed C1: 1u, Capacitors_SMD:C_0805, symbol C
- removed C2: 22n, Capacitors_SMD:C_0805, symbol C
- removed C3: 47u, Capacitors_SMD:C_0805, symbol C
- removed C5, C6: 22p, Capacitors_SMD:C_0805, symbol C
- removed L1: Ferrite bead, Resistors_SMD:R_0805, symbol Ferrite_Bead
- removed P1: USB_OTG, device.farm:conn_usb_B_micro_smd-2, symbol USB_OTG
- removed Q2, Q3: MMBT3904, TO_SOT_Packages_SMD:SOT-23, symbol MMBT3904
- removed R10, R11: 10k, Resistors_SMD:R_0805, symbol R
- removed R3, R4: 1k5, Resistors_SMD:R_0805, symbol R
- removed U1: RT9193, TO_SOT_Packages_SMD:SOT-23-5, symbol RT9193
- removed U5: CH340G, SMD_Packages:SO-16-N, symbol CH340G
- removed X1: 12MHz, Crystals:Crystal_SMD_SeikoEpson_TSX3225-4pin_3.2x2.5mm, symbol Crystal_GND24
- added X2: ESP-PROG, device.farm:Micro-Match-FOB-6, symbol ESP-PROG
- U2: value HLK-PM01 -> HLK-PM03; symbol HLK-PM01 -> HLK-PM03
- renumbered C8 to C1, C9 to C2, C4 to C3, C7 to C4, D1 to D2, R5 to R4, R6 to R5, R7 to R6, R8 to R7, R9 to R8, U4 to U3
Connections:
- net 5V is gone; now on net VCC: D2.3 (K)
- net 5V-USB is gone; now on net 3V3-MAINS: D2.1 (A)
- net GND: now also X2.1 (GND)
- net GPIO0: now also X2.4 (ESP_GPIO0)
- net MAINS-1: now also U2.1 (LINE1); no longer U2.2 (LINE2)
- net MAINS-2: now also U2.2 (LINE2); no longer U2.1 (LINE1)
- net RESET: now also X2.5 (ESP_RST)
- net RX: now also X2.3 (ESP_RX)
- net TX: now also X2.2 (ESP_TX)
- net 5V-MAINS renamed 3V3-MAINS
- net 3V3-MAINS: no longer D2.2 (A)
- new net 3V3-PROG: D2.2 (A), X2.6 (3V3)
- no-connect marks 6 -> 0
Other:
- moved on the sheet: C1, C2, C3, D2, U3
