File: board/SSR8A.kicad_pcb (KiCad board)
At the start: 2 copper layers, 155 x 55 mm, 55 parts, among them P1 USB_OTG, Q1 MMBT3904, Q2 MMBT3904, U1 PCF8574, U10 G3MB-SSR, U11 G3MB-SSR, U12 G3MB-SSR, U13 G3MB-SSR, U2 RT9193, U3 HLK-PM01, U4 ESP-12, U5 CH340G, U6 G3MB-SSR, U7 G3MB-SSR, U8 G3MB-SSR, U9 G3MB-SSR, X1 12MHz

Commit message: WIP
Parts:
- added C8: 47u, Capacitors_SMD:C_0805, F.Cu at (141.0, 110.0)
- added C9: 47u, Capacitors_SMD:C_0805, F.Cu at (141.0, 112.5)
- OUT1: renamed from  OUT1
- OUT2: renamed from  OUT2
- renumbered Q1 to Q2, Q2 to Q3, U2 to U1, U3 to U2, U1 to U3
Routing:
- net GND: track 51.4 -> 54.8 mm, vias 14 -> 16
- net VCC: track 119.4 -> 121.7 mm, vias 3 -> 4
Other:
- board text added: "Address"
- board text removed: "- stitek pro adresu - 2x47M vedle ESP"

Commit message: WIP
Parts:
- removed C6: 22p, Capacitors_SMD:C_0805
- removed C7: 100n, Capacitors_SMD:C_0805
- removed C8, C9: 47u, Capacitors_SMD:C_0805
- removed L1: Ferrite bead, Resistors_SMD:R_0805
- removed P1: USB_OTG, device.farm:conn_usb_B_micro_smd-2
- removed Q2, Q3: MMBT3904, TO_SOT_Packages_SMD:SOT-23
- removed R10, R11, R9: 10k, Resistors_SMD:R_0805
- removed R12, R13, R14, R15, R16, R17, R18, R19: 270R, Resistors_SMD:R_0805
- removed REF***: OSHW-Logo_11.4x12mm_SilkScreen, Symbols:OSHW-Logo_11.4x12mm_SilkScreen
- removed U12, U13: G3MB-SSR, device.farm:G3MB-SSR
- added D2: BAT54C, TO_SOT_Packages_SMD:SOT-23, F.Cu at (135.0, 155.9)
- added X2: ESP-PROG, device.farm:Micro-Match-FOB-6, F.Cu at (184.0, 100.0)
- C1: value 1u -> 47u
- C2: value 22n -> 47u
- C3: value 47u -> 100n
- C5: value 22p -> 100n
- D1: value BAT54C -> LED; footprint TO_SOT_Packages_SMD:SOT-23 -> LEDs:LED_0805
- IN1, OUT1, OUT2, OUT3, OUT4, OUT5, OUT6, OUT7, OUT8: footprint device.farm:DG301-5.0-02 -> device.farm:DG142R-2-5.08
- R1: value 4k7 -> 270R
- R3: value 1k5 -> 4k7
- R4: value 1k5 -> 10k
- U1: value RT9193 -> PCF8574; footprint TO_SOT_Packages_SMD:SOT-23-5 -> Housings_SOIC:SOIC-16W_7.5x10.3mm_Pitch1.27mm
- U2: value HLK-PM01 -> HLK-PM03
- U3: value PCF8574 -> ESP-12; footprint Housings_SOIC:SOIC-16W_7.5x10.3mm_Pitch1.27mm -> device.farm:ESP-12
- U4: value ESP-12 -> G3MB-SSR; footprint device.farm:ESP-12 -> device.farm:G3MB-SSR
- U5: value CH340G -> G3MB-SSR; footprint SMD_Packages:SO-16-N -> device.farm:G3MB-SSR
- X1: value 12MHz -> I2C; footprint Crystals:Crystal_SMD_SeikoEpson_TSX3225-4pin_3.2x2.5mm -> device.farm:Micro-Match-FOB-4
- moved U5 100.7 mm to (87.0, 124.5)
- moved U4 87.4 mm to (66.0, 124.5), turned to 270 degrees
- moved U3 79.6 mm to (204.5, 99.8), turned to 270 degrees
- moved C3 69.5 mm to (156.0, 155.0), turned to 0 degrees
- moved R8 66.3 mm to (178.1, 156.0), turned to 0 degrees
- moved U11 65.7 mm to (213.0, 124.5)
- moved C2 63.4 mm to (148.0, 156.0)
- moved U10 62.2 mm to (192.0, 124.5)
- moved X1 62.0 mm to (117.0, 100.0)
- moved R7 61.5 mm to (178.1, 153.0), turned to 0 degrees
- moved C4 60.3 mm to (152.0, 152.0), turned to 0 degrees
- moved U9 58.8 mm to (171.0, 124.5)
- moved R2 58.2 mm to (162.9, 155.0), turned to 0 degrees
- moved C1 57.3 mm to (127.0, 154.0), turned to 0 degrees
- moved U8 55.3 mm to (150.0, 124.5)
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Connections:
- C1 pad 1: /5V -> VCC
- C2 pad 1: Net-(C2-Pad1) -> VCC
- C3 pad 1: Net-(C3-Pad1) -> VCC
- C4 pad 1: VCC -> GND
- C4 pad 2: GND -> /ESP/RESET
- C5 pad 1: Net-(C5-Pad1) -> VCC
- D1 pad 1: /ESP/5V-USB -> GND
- D1 pad 2: /ESP/5V-MAINS -> Net-(D1-Pad2)
- R1 pad 1: VCC -> Net-(D1-Pad2)
- R1 pad 2: /SDA -> /ESP/GPIO4
- R2 pad 1: /SCL -> VCC
- R2 pad 2: VCC -> /SDA
- R3 pad 1: /ESP/RX -> /SCL
- R3 pad 2: Net-(R3-Pad2) -> VCC
- R4 pad 1: /ESP/TX -> /ESP/GPIO0
- R4 pad 2: Net-(R4-Pad2) -> VCC
- R5 pad 1: /ESP/GPIO0 -> /ESP/GPIO2
- R6 pad 1: /ESP/GPIO2 -> /ESP/EN
- R7 pad 1: /ESP/EN -> /ESP/RESET
- R8 pad 1: /ESP/RESET -> /ESP/GPIO15
- R8 pad 2: VCC -> GND
- U1 pad 1: /5V -> GND
- U1 pad 3: /5V -> GND
- U1 pad 4: Net-(C2-Pad1) -> /ssr-channel-0//SW
- U1 pad 5: Net-(C3-Pad1) -> /ssr-channel-1//SW
- U10 pad 2: Net-(OUT5-Pad1) -> Net-(OUT7-Pad1)
- U10 pad 3: Net-(R16-Pad1) -> VCC
- U10 pad 4: /ssr-channel-4//SW -> /ssr-channel-6//SW
- U11 pad 2: Net-(OUT6-Pad1) -> Net-(OUT8-Pad1)
- U11 pad 3: Net-(R17-Pad1) -> VCC
- U11 pad 4: /ssr-channel-5//SW -> /ssr-channel-7//SW
- U2 pad 1: /MAINS-N -> /MAINS-L
- U2 pad 2: /MAINS-L -> /MAINS-N
- U2 pad 4: /ESP/5V-MAINS -> /ESP/3V3-MAINS
- U3 pad 1: GND -> /ESP/RESET
- U3 pad 10: /ssr-channel-5//SW -> /ESP/GPIO15
- U3 pad 11: /ssr-channel-6//SW -> /ESP/GPIO2
- U3 pad 12: /ssr-channel-7//SW -> /ESP/GPIO0
- U3 pad 13: (no net) -> /ESP/GPIO4
- U3 pad 14: /SCL -> (no net)
- U3 pad 15: /SDA -> /ESP/RX
- U3 pad 16: VCC -> /ESP/TX
- U3 pad 2: GND -> (no net)
- U3 pad 3: GND -> /ESP/EN
- U3 pad 4: /ssr-channel-0//SW -> (no net)
- U3 pad 5: /ssr-channel-1//SW -> /SCL
- U3 pad 6: /ssr-channel-2//SW -> /SDA
- U3 pad 7: /ssr-channel-3//SW -> (no net)
- U3 pad 8: GND -> VCC
- U3 pad 9: /ssr-channel-4//SW -> GND
- U4 pad 1: /ESP/RESET -> /MAINS-L
- U4 pad 2: (no net) -> Net-(OUT1-Pad1)
- U4 pad 3: /ESP/EN -> VCC
- U4 pad 4: (no net) -> /ssr-channel-0//SW
- U5 pad 1: GND -> /MAINS-L
- U5 pad 2: Net-(R3-Pad2) -> Net-(OUT2-Pad1)
- U5 pad 3: Net-(R4-Pad2) -> VCC
- U5 pad 4: VCC -> /ssr-channel-1//SW
- U6 pad 2: Net-(OUT1-Pad1) -> Net-(OUT3-Pad1)
- U6 pad 3: Net-(R12-Pad1) -> VCC
- U6 pad 4: /ssr-channel-0//SW -> /ssr-channel-2//SW
- U7 pad 2: Net-(OUT2-Pad1) -> Net-(OUT4-Pad1)
- U7 pad 3: Net-(R13-Pad1) -> VCC
- U7 pad 4: /ssr-channel-1//SW -> /ssr-channel-3//SW
- U8 pad 2: Net-(OUT3-Pad1) -> Net-(OUT5-Pad1)
- U8 pad 3: Net-(R14-Pad1) -> VCC
- U8 pad 4: /ssr-channel-2//SW -> /ssr-channel-4//SW
- U9 pad 2: Net-(OUT4-Pad1) -> Net-(OUT6-Pad1)
- U9 pad 3: Net-(R15-Pad1) -> VCC
- U9 pad 4: /ssr-channel-3//SW -> /ssr-channel-5//SW
- X1 pad 1: Net-(C5-Pad1) -> GND
- X1 pad 2: GND -> /SCL
- X1 pad 3: Net-(C6-Pad1) -> /SDA
- X1 pad 4: GND -> VCC
Routing:
- net /MAINS-N: track 212.8 -> 0.00 mm
- net /MAINS-L: track 179.5 -> 0.00 mm
- net /5V: track 166.2 -> 0.00 mm, vias 9 -> 0
- net /ESP/5V-USB: track 129.5 -> 0.00 mm, vias 4 -> 0
- net VCC: track 121.7 -> 0.00 mm, vias 4 -> 0
- net /ssr-channel-0//SW: track 67.3 -> 0.00 mm
- net /ESP/RESET: track 59.8 -> 0.00 mm
- net /ssr-channel-7//SW: track 56.9 -> 0.00 mm
- net GND: track 54.8 -> 0.00 mm, vias 16 -> 0
- net /ssr-channel-1//SW: track 47.6 -> 0.00 mm
- net /ssr-channel-6//SW: track 38.9 -> 0.00 mm
- net /ESP/GPIO0: track 38.6 -> 0.00 mm, vias 2 -> 0
- net /ssr-channel-2//SW: track 29.6 -> 0.00 mm
- net /SCL: track 24.7 -> 0.00 mm
- net /ssr-channel-5//SW: track 20.8 -> 0.00 mm
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- removed copper zone on B.Cu, net GND
Other:
- board size 155 x 55 mm -> 182 x 48 mm
- net class Default: trace_width 0.4 -> 0.25
- board text removed: "1"
- board text removed: "100-240VAC"
- board text removed: "2"
- board text removed: "3"
- board text removed: "4"
- board text removed: "400W max."
- board text removed: "5"
- board text removed: "6"
- board text removed: "7"
- board text removed: "8"
- board text removed: "Address"
- board text removed: "CC-BY-SA"
- board text removed: "DEVICE.FARM"
- board text removed: "IN"
- board text removed: "L"
- board text removed: "N"
- board text removed: "SSR8A 1.0"

Commit message: WIP
Parts:
- added REF***: OSHW-Logo_11.4x12mm_SilkScreen, Symbols:OSHW-Logo_11.4x12mm_SilkScreen, F.Cu at (153.5, 101.0)
- moved C1 85.6 mm to (186.0, 92.0), turned to 90 degrees
- moved D1 82.6 mm to (180.9, 101.0)
- moved C2 75.5 mm to (188.0, 92.0), turned to 90 degrees
- moved C3 71.6 mm to (190.0, 92.0), turned to 90 degrees
- moved D2 69.2 mm to (162.5, 92.5)
- moved C4 65.7 mm to (188.0, 97.0)
- moved R6 62.8 mm to (187.9, 95.0), turned to 180 degrees
- moved R2 61.9 mm to (143.9, 96.0), turned to 270 degrees
- moved R1 55.9 mm to (187.9, 101.0)
- moved R3 55.1 mm to (144.0, 101.0), turned to 270 degrees
- moved R7 54.9 mm to (187.9, 99.0), turned to 180 degrees
- moved R4 54.7 mm to (187.9, 103.0), turned to 180 degrees
- moved R8 50.0 mm to (187.9, 107.0), turned to 180 degrees
- moved R5 50.0 mm to (187.9, 105.0), turned to 180 degrees
- moved U3 12.0 mm to (192.5, 99.8)
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Routing:
- net VCC: track 0.00 -> 331.7 mm, vias 0 -> 2
- net /MAINS-N: track 0.00 -> 303.4 mm
- net /MAINS-L: track 0.00 -> 202.3 mm
- net /SDA: track 0.00 -> 103.5 mm, vias 0 -> 3
- net /SCL: track 0.00 -> 103.4 mm, vias 0 -> 3
- net /ssr-channel-7//SW: track 0.00 -> 81.4 mm
- net /ESP/3V3-MAINS: track 0.00 -> 75.6 mm
- net /ssr-channel-0//SW: track 0.00 -> 69.6 mm
- net /ssr-channel-6//SW: track 0.00 -> 60.3 mm
- net /ssr-channel-1//SW: track 0.00 -> 48.8 mm
- net /ESP/TX: track 0.00 -> 47.4 mm, vias 0 -> 2
- net /ESP/RESET: track 0.00 -> 44.3 mm, vias 0 -> 2
- net /ESP/GPIO0: track 0.00 -> 40.2 mm, vias 0 -> 2
- net /ssr-channel-5//SW: track 0.00 -> 38.2 mm
- net /ESP/RX: track 0.00 -> 35.9 mm, vias 0 -> 2
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- added copper zone on B.Cu, net GND
Other:
- outline, holes or cut-outs redrawn
- net class Default: trace_width 0.25 -> 0.4
- board text added: "0"
- board text added: "1"
- board text added: "100-240V"
- board text added: "2"
- board text added: "3"
- board text added: "4"
- board text added: "5"
- board text added: "6"
- board text added: "7"
- board text added: "Address"
- board text added: "CHANNEL"
- board text added: "DEVICE.FARM SSR v1.0 CC-BY-SA Max load: 2A / channel"
- board text added: "ESPP"
- board text added: "I2C"
- board text added: "MAINS"

Commit message: WIP
Other:
- board text added: "DEVICE.FARM SSR8A v1.0 CC-BY-SA Max load: 2A/channel"
- board text removed: "DEVICE.FARM SSR v1.0 CC-BY-SA Max load: 2A / channel"
Changed lines of the file:
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@@
   )
   (gr_line (start 102.5 92.5) (end 159 92.5) (layer F.SilkS) (width 0.2))
-  (gr_text "DEVICE.FARM   SSR v1.0   CC-BY-SA   Max load: 2A / channel" (at 130.5 91) (layer F.SilkS)
+  (gr_text "DEVICE.FARM   SSR8A v1.0   CC-BY-SA   Max load: 2A/channel" (at 130.5 91) (layer F.SilkS)
     (effects (font (size 1.1 1.1) (thickness 0.275)))
   )
