File: board/SSR8A.kicad_pcb (KiCad board)
At the start: 2 copper layers, 182 x 48 mm, 38 parts, among them U1 PCF8574, U10 G3MB-SSR, U11 G3MB-SSR, U2 HLK-PM03, U3 ESP-12, U4 G3MB-SSR, U5 G3MB-SSR, U6 G3MB-SSR, U7 G3MB-SSR, U8 G3MB-SSR, U9 G3MB-SSR, X1 I2C, X2 ESP-PROG

Commit message: WIP
Parts:
- removed C4, C5: 100n, Capacitors_SMD:C_0805
- removed D2: BAT54C, TO_SOT_Packages_SMD:SOT-23
- removed OUT1, OUT2, OUT3, OUT4, OUT5, OUT6, OUT7, OUT8: Conn_01x02, device.farm:DG142R-2-5.08
- removed R4, R5, R6, R7, R8: 10k, Resistors_SMD:R_0805
- removed REF***: OSHW-Logo_11.4x12mm_SilkScreen, Symbols:OSHW-Logo_11.4x12mm_SilkScreen
- added J1: Conn_01x02, Drake:DG235-3.81-02P, F.Cu at (74.7, 114.8)
- added J2: Conn_01x02, Drake:DG235-3.81-02P, F.Cu at (95.7, 114.8)
- added J3: Conn_01x02, Drake:DG235-3.81-02P, F.Cu at (116.7, 114.8)
- added J4: Conn_01x02, Drake:DG235-3.81-02P, F.Cu at (137.7, 114.8)
- added J5: Conn_01x02, Drake:DG235-3.81-02P, F.Cu at (158.7, 114.8)
- added J6: Conn_01x02, Drake:DG235-3.81-02P, F.Cu at (179.7, 114.8)
- added J7: Conn_01x02, Drake:DG235-3.81-02P, F.Cu at (200.7, 114.8)
- added J8: Conn_01x02, Drake:DG235-3.81-02P, F.Cu at (221.7, 114.8)
- added J9: PROG, Connector_PinHeader_2.54mm:PinHeader_1x03_P2.54mm_Vertical, F.Cu at (189.0, 91.5)
- added RV1: B72650M251K72, Resistor_SMD:R_1210_3225Metric_Pad1.30x2.65mm_HandSolder, F.Cu at (56.6, 109.0)
- added X3: I2C, Connector_IDC:IDC-Header_2x03_P2.54mm_Vertical, F.Cu at (149.2, 95.5)
- C1, C2: value 47u -> C; footprint Capacitors_SMD:C_0805 -> Capacitor_SMD:C_0805_2012Metric_Pad1.18x1.45mm_HandSolder
- C3: value 100n -> C; footprint Capacitors_SMD:C_0805 -> Capacitor_SMD:C_0805_2012Metric_Pad1.18x1.45mm_HandSolder
- D1: footprint LEDs:LED_0805 -> LED_SMD:LED_0805_2012Metric_Pad1.15x1.40mm_HandSolder
- IN1: footprint device.farm:DG142R-2-5.08 -> Drake:DG235-3.81-02P
- R1: value 270R -> 4k7; footprint Resistors_SMD:R_0805 -> Resistor_SMD:R_0805_2012Metric_Pad1.20x1.40mm_HandSolder
- R2: footprint Resistors_SMD:R_0805 -> Resistor_SMD:R_0805_2012Metric_Pad1.20x1.40mm_HandSolder
- R3: value 4k7 -> 270R; footprint Resistors_SMD:R_0805 -> Resistor_SMD:R_0805_2012Metric_Pad1.20x1.40mm_HandSolder
- U1: value PCF8574 -> LM1117-3.3; footprint Housings_SOIC:SOIC-16W_7.5x10.3mm_Pitch1.27mm -> Package_TO_SOT_SMD:SOT-223-3_TabPin2
- U10, U11, U4, U5, U6, U7, U8, U9: footprint device.farm:G3MB-SSR -> Drake:G3MB-SSR
- U2: value HLK-PM03 -> HLK-PM01; footprint device.farm:HLK-PM01 -> Drake:HLK-PM01
- U3: value ESP-12 -> ESP32-C3-WROOM-02; footprint device.farm:ESP-12 -> Espressif:ESP32-C3-WROOM-02
- X1: footprint device.farm:Micro-Match-FOB-4 -> Drake:Micro-Match-FOB-4
- X2: value ESP-PROG -> I2C; footprint device.farm:Micro-Match-FOB-6 -> Drake:Micro-Match-FOB-6
- moved C1 65.7 mm to (120.5, 97.0)
- moved X1 64.2 mm to (176.0, 95.0)
- moved C2 54.3 mm to (134.0, 98.0)
- moved C3 53.3 mm to (137.0, 98.0)
- moved R1 45.5 mm to (142.5, 98.0), turned to 180 degrees
- moved R3 43.5 mm to (187.5, 102.0), turned to 0 degrees
- moved U3 13.6 mm to (206.0, 101.0), turned to 0 degrees
- moved X2 7.81 mm to (166.0, 95.0)
- moved U1 6.77 mm to (127.5, 98.0)
- moved IN1 4.70 mm to (54.7, 114.8)
- moved D1 2.33 mm to (183.0, 102.0)
- moved R2 1.55 mm to (142.5, 95.5), turned to 0 degrees
Connections:
- C1 pad 1: VCC -> +5V
- C2 pad 1: VCC -> +3V3
- C3 pad 1: VCC -> +3V3
- D1 pad 2: Net-(D1-Pad2) -> Net-(D1-A)
- R1 pad 1: Net-(D1-Pad2) -> /SDA
- R1 pad 2: /ESP/GPIO4 -> +5V
- R2 pad 1: VCC -> +5V
- R2 pad 2: /SDA -> /SCL
- R3 pad 1: /SCL -> Net-(D1-A)
- R3 pad 2: VCC -> /LED
- U1 pad 2: GND -> +3V3
- U1 pad 3: GND -> +5V
- U10 pad 3: VCC -> +5V
- U10 pad 4: /ssr-channel-6//SW -> //CH6
- U11 pad 3: VCC -> +5V
- U11 pad 4: /ssr-channel-7//SW -> //CH7
- U2 pad 4: /ESP/3V3-MAINS -> +5V
- U3 pad 1: /ESP/RESET -> +3V3
- U3 pad 10: /ESP/GPIO15 -> //CH5
- U3 pad 11: /ESP/GPIO2 -> //CH6
- U3 pad 12: /ESP/GPIO0 -> //CH7
- U3 pad 13: /ESP/GPIO4 -> /USB_D-
- U3 pad 14: (no net) -> /USB_D+
- U3 pad 15: /ESP/RX -> /SCL
- U3 pad 16: /ESP/TX -> /SDA
- U3 pad 2: (no net) -> +3V3
- U3 pad 3: /ESP/EN -> //CH0
- U3 pad 4: (no net) -> //CH1
- U3 pad 5: /SCL -> //CH2
- U3 pad 6: /SDA -> //CH3
- U3 pad 7: (no net) -> //CH4
- U3 pad 8: VCC -> unconnected-(U3-GPIO9)
- U4 pad 3: VCC -> +5V
- U4 pad 4: /ssr-channel-0//SW -> //CH0
- U5 pad 3: VCC -> +5V
- U5 pad 4: /ssr-channel-1//SW -> //CH1
- U6 pad 3: VCC -> +5V
- U6 pad 4: /ssr-channel-2//SW -> //CH2
- U7 pad 3: VCC -> +5V
- U7 pad 4: /ssr-channel-3//SW -> //CH3
- U8 pad 3: VCC -> +5V
- U8 pad 4: /ssr-channel-4//SW -> //CH4
- U9 pad 3: VCC -> +5V
- U9 pad 4: /ssr-channel-5//SW -> //CH5
- X1 pad 4: VCC -> +3V3
- X2 pad 2: /ESP/TX -> /SCL
- X2 pad 3: /ESP/RX -> /SDA
- X2 pad 4: /ESP/GPIO0 -> +3V3
- X2 pad 5: /ESP/RESET -> +5V
- X2 pad 6: /ESP/3V3-PROG -> /ALERT
Routing:
- net VCC: track 331.7 -> 0.00 mm, vias 2 -> 0
- net +5V: track 0.00 -> 282.1 mm, vias 0 -> 1
- net //CH0: track 0.00 -> 138.0 mm
- net //CH1: track 0.00 -> 116.9 mm
- net //CH2: track 0.00 -> 95.6 mm
- net +3V3: track 0.00 -> 95.1 mm
- net /ssr-channel-7//SW: track 81.4 -> 0.00 mm
- net /ESP/3V3-MAINS: track 75.6 -> 0.00 mm
- net //CH3: track 0.00 -> 73.7 mm
- net /ssr-channel-0//SW: track 69.6 -> 0.00 mm
- net /ALERT: track 0.00 -> 69.2 mm, vias 0 -> 4
- net /ssr-channel-6//SW: track 60.3 -> 0.00 mm
- net //CH4: track 0.00 -> 52.1 mm
- net /ssr-channel-1//SW: track 48.8 -> 0.00 mm
- net /ESP/TX: track 47.4 -> 0.00 mm, vias 2 -> 0
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Other:
- outline, holes or cut-outs redrawn
- net class Default removed
- board text added: "SSR8A v2.0 CC-BY-SA Max load: 2A/channel"
- board text removed: "Address"
- board text removed: "DEVICE.FARM SSR8A v1.0 CC-BY-SA Max load: 2A/channel"
- board text removed: "ESPP"
- board text removed: "I2C"

Commit message: WIP
Parts:
- added H1: MountingHole, MountingHole:MountingHole_3.7mm_Pad_Via, F.Cu at (109.0, 95.0)
Changed lines of the file:
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@@
 (kicad_pcb (version 20221018) (generator pcbnew)
   (general
-    (thickness 1.58)
+    (thickness 1.6)
   )
   (paper "A4")
@@
   (setup
     (stackup
+      (layer "F.SilkS" (type "Top Silk Screen") (color "White"))
+      (layer "F.Paste" (type "Top Solder Paste"))
+      (layer "F.Mask" (type "Top Solder Mask") (color "Black") (thickness 0.01))
       (layer "F.Cu" (type "copper") (thickness 0.035))
       (layer "dielectric 1" (type "core") (thickness 1.51) (material "FR4") (epsilon_r 4.5) (loss_tangent 0.02))
       (layer "B.Cu" (type "copper") (thickness 0.035))
+      (layer "B.Mask" (type "Bottom Solder Mask") (color "Black") (thickness 0.01))
+      (layer "B.Paste" (type "Bottom Solder Paste"))
+      (layer "B.SilkS" (type "Bottom Silk Screen") (color "White"))
       (copper_finish "None")
       (dielectric_constraints no)
@@
     (fp_line (start 1 0.625) (end -1 0.625)
       (stroke (width 0.1) (type solid)) (layer "F.Fab"))
-    (pad "1" smd roundrect (at -1.0375 0 90) (size 1.175 1.45) (layers "F.Cu" "F.Paste" "F.Mask") (roundrect_rratio 0.212766)
+    (pad "1" smd roundrect (at -1.0375 0 90) (size 1.175 1.45) (layers "F.Cu" "F.Paste" "F.Mask") (roundrect_rratio 0.2127659574)
       (net 6 "+5V") (pintype "passive"))
-    (pad "2" smd roundrect (at 1.0375 0 90) (size 1.175 1.45) (layers "F.Cu" "F.Paste" "F.Mask") (roundrect_rratio 0.212766)
+    (pad "2" smd roundrect (at 1.0375 0 90) (size 1.175 1.45) (layers "F.Cu" "F.Paste" "F.Mask") (roundrect_rratio 0.2127659574)
       (net 1 "GND") (pintype "passive"))
     (model "${KICAD6_3DMODEL_DIR}/Capacitor_SMD.3dshapes/C_0805_2012Metric.wrl"
@@
     (fp_line (start 1 0.625) (end -1 0.625)
       (stroke (width 0.1) (type solid)) (layer "F.Fab"))
-    (pad "1" smd roundrect (at -1.0375 0 90) (size 1.175 1.45) (layers "F.Cu" "F.Paste" "F.Mask") (roundrect_rratio 0.212766)
+    (pad "1" smd roundrect (at -1.0375 0 90) (size 1.175 1.45) (layers "F.Cu" "F.Paste" "F.Mask") (roundrect_rratio 0.2127659574)
       (net 7 "+3V3") (pintype "passive"))
-    (pad "2" smd roundrect (at 1.0375 0 90) (size 1.175 1.45) (layers "F.Cu" "F.Paste" "F.Mask") (roundrect_rratio 0.212766)
+    (pad "2" smd roundrect (at 1.0375 0 90) (size 1.175 1.45) (layers "F.Cu" "F.Paste" "F.Mask") (roundrect_rratio 0.2127659574)
       (net 1 "GND") (pintype "passive"))
     (model "${KICAD6_3DMODEL_DIR}/Capacitor_SMD.3dshapes/C_0805_2012Metric.wrl"
@@
     (fp_line (start 1 0.625) (end -1 0.625)
       (stroke (width 0.1) (type solid)) (layer "F.Fab"))
-    (pad "1" smd roundrect (at -1.0375 0 90) (size 1.175 1.45) (layers "F.Cu" "F.Paste" "F.Mask") (roundrect_rratio 0.212766)
+    (pad "1" smd roundrect (at -1.0375 0 90) (size 1.175 1.45) (layers "F.Cu" "F.Paste" "F.Mask") (roundrect_rratio 0.2127659574)
       (net 7 "+3V3") (pintype "passive"))
-    (pad "2" smd roundrect (at 1.0375 0 90) (size 1.175 1.45) (layers "F.Cu" "F.Paste" "F.Mask") (roundrect_rratio 0.212766)
+    (pad "2" smd roundrect (at 1.0375 0 90) (size 1.175 1.45) (layers "F.Cu" "F.Paste" "F.Mask") (roundrect_rratio 0.2127659574)
       (net 1 "GND") (pintype "passive"))
     (model "${KICAD6_3DMODEL_DIR}/Capacitor_SMD.3dshapes/C_0805_2012Metric.wrl"
@@
     (fp_line (start 1 0.6) (end 1 -0.6)
       (stroke (width 0.1) (type solid)) (layer "F.Fab"))
-    (pad "1" smd roundrect (at -1.025 0) (size 1.15 1.4) (layers "F.Cu" "F.Paste" "F.Mask") (roundrect_rratio 0.217391)
+    (pad "1" smd roundrect (at -1.025 0) (size 1.15 1.4) (layers "F.Cu" "F.Paste" "F.Mask") (roundrect_rratio 0.2173913043)
       (net 1 "GND") (pinfunction "K") (pintype "passive"))
-    (pad "2" smd roundrect (at 1.025 0) (size 1.15 1.4) (layers "F.Cu" "F.Paste" "F.Mask") (roundrect_rratio 0.217391)
+    (pad "2" smd roundrect (at 1.025 0) (size 1.15 1.4) (layers "F.Cu" "F.Paste" "F.Mask") (roundrect_rratio 0.2173913043)
       (net 8 "Net-(D1-A)") (pinfunction "A") (pintype "passive"))
     (model "${KICAD6_3DMODEL_DIR}/LED_SMD.3dshapes/LED_0805_2012Metric.wrl"
@@
     (fp_line (start 1 0.625) (end -1 0.625)
       (stroke (width 0.1) (type solid)) (layer "F.Fab"))
-    (pad "1" smd roundrect (at -1 0 180) (size 1.2 1.4) (layers "F.Cu" "F.Paste" "F.Mask") (roundrect_rratio 0.208333)
+    (pad "1" smd roundrect (at -1 0 180) (size 1.2 1.4) (layers "F.Cu" "F.Paste" "F.Mask") (roundrect_rratio 0.2083333333)
       (net 4 "/SDA") (pintype "passive"))
-    (pad "2" smd roundrect (at 1 0 180) (size 1.2 1.4) (layers "F.Cu" "F.Paste" "F.Mask") (roundrect_rratio 0.208333)
+    (pad "2" smd roundrect (at 1 0 180) (size 1.2 1.4) (layers "F.Cu" "F.Paste" "F.Mask") (roundrect_rratio 0.2083333333)
       (net 6 "+5V") (pintype "passive"))
     (model "${KICAD6_3DMODEL_DIR}/Resistor_SMD.3dshapes/R_0805_2012Metric.wrl"
@@
     (fp_line (start 1 0.625) (end -1 0.625)
       (stroke (width 0.1) (type solid)) (layer "F.Fab"))
-    (pad "1" smd roundrect (at -1 0) (size 1.2 1.4) (layers "F.Cu" "F.Paste" "F.Mask") (roundrect_rratio 0.208333)
+    (pad "1" smd roundrect (at -1 0) (size 1.2 1.4) (layers "F.Cu" "F.Paste" "F.Mask") (roundrect_rratio 0.2083333333)
       (net 6 "+5V") (pintype "passive"))
-    (pad "2" smd roundrect (at 1 0) (size 1.2 1.4) (layers "F.Cu" "F.Paste" "F.Mask") (roundrect_rratio 0.208333)
+    (pad "2" smd roundrect (at 1 0) (size 1.2 1.4) (layers "F.Cu" "F.Paste" "F.Mask") (roundrect_rratio 0.2083333333)
       (net 5 "/SCL") (pintype "passive"))
     (model "${KICAD6_3DMODEL_DIR}/Resistor_SMD.3dshapes/R_0805_2012Metric.wrl"
@@
     (fp_line (start 1 0.625) (end -1 0.625)
       (stroke (width 0.1) (type solid)) (layer "F.Fab"))
-    (pad "1" smd roundrect (at -1 0) (size 1.2 1.4) (layers "F.Cu" "F.Paste" "F.Mask") (roundrect_rratio 0.208333)
+    (pad "1" smd roundrect (at -1 0) (size 1.2 1.4) (layers "F.Cu" "F.Paste" "F.Mask") (roundrect_rratio 0.2083333333)
       (net 8 "Net-(D1-A)") (pintype "passive"))
-    (pad "2" smd roundrect (at 1 0) (size 1.2 1.4) (layers "F.Cu" "F.Paste" "F.Mask") (roundrect_rratio 0.208333)
+    (pad "2" smd roundrect (at 1 0) (size 1.2 1.4) (layers "F.Cu" "F.Paste" "F.Mask") (roundrect_rratio 0.2083333333)
       (net 19 "/LED") (pintype "passive"))
     (model "${KICAD6_3DMODEL_DIR}/Resistor_SMD.3dshapes/R_0805_2012Metric.wrl"
@@
     (pad "3" thru_hole oval (at 0 5.08 270) (size 1.7 1.7) (drill 1) (layers *.Cu *.Mask)
       (net 18 "/USB_D-") (pinfunction "Pin_3") (pintype "passive"))
-    (model "${KICAD6_3DMODEL_DIR}/Connector_PinHeader_2.54mm.3dshapes/PinHeader_1x03_P2.54mm_Vertical.wrl"
+    (model "${KICAD6_3DMODEL_DIR}/Connector_PinHeader_2.54mm.3dshapes/PinHeader_1x03_P2.54mm_Vertical.wrl" hide
       (offset (xyz 0 0 0))
       (scale (xyz 1 1 1))
@@
     (fp_line (start 5.72 10.18) (end -3.18 10.18)
       (stroke (width 0.1) (type solid)) (layer "F.Fab"))
-    (pad "1" thru_hole roundrect (at 0 0) (size 1.7 1.7) (drill 1) (layers *.Cu *.Mask) (roundrect_rratio 0.147059)
+    (pad "1" thru_hole roundrect (at 0 0) (size 1.7 1.7) (drill 1) (layers *.Cu *.Mask) (roundrect_rratio 0.1470588235)
       (net 1 "GND") (pinfunction "GND") (pintype "power_in"))
     (pad "2" thru_hole circle (at 2.54 0) (size 1.7 1.7) (drill 1) (layers *.Cu *.Mask)
@@
     )
   )
+  (footprint "MountingHole:MountingHole_3.7mm_Pad_Via" (layer "F.Cu")
+    (at 109 95)
+    (descr "Mounting Hole 3.7mm")
+    (tags "mounting hole 3.7mm")
+    (property "Sheetfile" "SSR8A.kicad_sch")
+    (property "Sheetname" "")
+    (property "ki_description" "Mounting Hole without connection")
+    (property "ki_keywords" "mounting hole")
+    (fp_text reference "H1" (at 0 -4.7) (layer "F.SilkS") hide
+        (effects (font (size 1 1) (thickness 0.15)))
+    )
+    (fp_text value "MountingHole" (at 0 4.7) (layer "F.Fab")
+        (effects (font (size 1 1) (thickness 0.15)))
+    )
+    (fp_text user "${REFERENCE}" (at 0 0) (layer "F.Fab")
+        (effects (font (size 1 1) (thickness 0.15)))
+    )
+    (fp_circle (center 0 0) (end 3.7 0)
+      (stroke (width 0.15) (type solid)) (fill none) (layer "Cmts.User"))
+    (fp_circle (center 0 0) (end 3.95 0)
+      (stroke (width 0.05) (type solid)) (fill none) (layer "F.CrtYd"))
+    (pad "1" thru_hole circle (at -2.775 0) (size 0.8 0.8) (drill 0.5) (layers *.Cu *.Mask))
+    (pad "1" thru_hole circle (at -1.962221 -1.962221) (size 0.8 0.8) (drill 0.5) (layers *.Cu *.Mask))
+    (pad "1" thru_hole circle (at -1.962221 1.962221) (size 0.8 0.8) (drill 0.5) (layers *.Cu *.Mask))
+    (pad "1" thru_hole circle (at 0 -2.775) (size 0.8 0.8) (drill 0.5) (layers *.Cu *.Mask))
+    (pad "1" thru_hole circle (at 0 0) (size 7.4 7.4) (drill 3.7) (layers *.Cu *.Mask))
+    (pad "1" thru_hole circle (at 0 2.775) (size 0.8 0.8) (drill 0.5) (layers *.Cu *.Mask))
+    (pad "1" thru_hole circle (at 1.962221 -1.962221) (size 0.8 0.8) (drill 0.5) (layers *.Cu *.Mask))
+    (pad "1" thru_hole circle (at 1.962221 1.962221) (size 0.8 0.8) (drill 0.5) (layers *.Cu *.Mask))
+    (pad "1" thru_hole circle (at 2.775 0) (size 0.8 0.8) (drill 0.5) (layers *.Cu *.Mask))
+  )
   (footprint "Drake:DG235-3.81-02P" locked (layer "F.Cu")
     (at 221.73 114.825)
@@
     (fp_line (start 1.6 1.245) (end -1.6 1.245)
       (stroke (width 0.1) (type solid)) (layer "F.Fab"))
-    (pad "1" smd roundrect (at -1.55 0) (size 1.3 2.65) (layers "F.Cu" "F.Paste" "F.Mask") (roundrect_rratio 0.192308)
+    (pad "1" smd roundrect (at -1.55 0) (size 1.3 2.65) (layers "F.Cu" "F.Paste" "F.Mask") (roundrect_rratio 0.1923076923)
       (net 2 "/MAINS-L") (pintype "passive"))
-    (pad "2" smd roundrect (at 1.55 0) (size 1.3 2.65) (layers "F.Cu" "F.Paste" "F.Mask") (roundrect_rratio 0.192308)
+    (pad "2" smd roundrect (at 1.55 0) (size 1.3 2.65) (layers "F.Cu" "F.Paste" "F.Mask") (roundrect_rratio 0.1923076923)
       (net 3 "/MAINS-N") (pintype "passive"))
     (model "${KICAD6_3DMODEL_DIR}/Resistor_SMD.3dshapes/R_1210_3225Metric.wrl"

Commit message: WIP
Parts:
- added C1: 1u, Capacitor_SMD:C_0805_2012Metric_Pad1.18x1.45mm_HandSolder, F.Cu at (192.2, 100.0)
- added R4: 10k, Resistor_SMD:R_0805_2012Metric_Pad1.20x1.40mm_HandSolder, F.Cu at (194.5, 97.8)
- C2: renamed from C1; value C -> 10u
- C3: renamed from C2; value C -> 47u
- C4: renamed from C3; value C -> 47u
- renumbered J9 to J1, J1 to J2, J2 to J3, J3 to J4, J4 to J5, J5 to J6, J6 to J7, J7 to J8, J8 to J9, R3 to R1, R1 to R2, R2 to R3, U2 to U1, U3 to U2, U1 to U3
Connections:
- U2 pad 2: +3V3 -> Net-(U2-EN/CHIP_PU)
Routing:
- net Net-(U2-EN/CHIP_PU): track 0.00 -> 5.25 mm
- net GND: track 28.7 -> 32.2 mm, vias 21 -> 22
- net +3V3: track 95.1 -> 93.6 mm
- net /SCL: track 79.8 -> 81.0 mm
- net /SDA: track 76.0 -> 76.9 mm
- net /USB_D+: track 31.9 -> 32.6 mm

Commit message: WIP
Other:
- board text added: "SSR8A v2.1 drake.cz Max load: 2A/channel"
- board text removed: "SSR8A v2.0 CC-BY-SA Max load: 2A/channel"

Commit message: WIP
Parts:
- U2: footprint Espressif:ESP32-C3-WROOM-02 -> Drake:ESP32-C3-WROOM-02 Handsolder
- moved D1 3.47 mm to (179.5, 102.0)
- moved R1 3.47 mm to (184.0, 102.0)
- moved C1 2.75 mm to (189.5, 100.0)
- moved R4 2.50 mm to (192.0, 97.8)
Routing:
- net GND: track 32.2 -> 3.83 mm, vias 22 -> 78
- net /LED: track 27.8 -> 31.7 mm
- net //CH7: track 11.7 -> 14.0 mm
- net Net-(U2-EN/CHIP_PU): track 5.25 -> 7.50 mm
- net //CH6: track 31.9 -> 33.7 mm
- net /SCL: track 81.0 -> 79.7 mm
- net //CH5: track 47.2 -> 47.7 mm
- net //CH4: track 52.1 -> 51.6 mm
- net //CH2: track 95.6 -> 95.1 mm
- net //CH1: track 116.9 -> 116.4 mm
- net /USB_D-: track 37.6 -> 38.1 mm
- net /USB_D+: track 32.6 -> 33.1 mm
- net /ALERT: track 69.2 -> 69.7 mm
- added copper zone on F.Cu, net GND
