File: board/SSR8A.kicad_sch (KiCad schematic)
At the start: 16 parts, among them J2 PROG, U1 LM1117-3.3, U2 HLK-PM01, U3 ESP32-C3-WROOM-02, X1 I2C, X2 I2C, X3 I2C

Commit message: WIP
Parts:
- added H1: MountingHole, MountingHole:MountingHole_3.7mm_Pad_Via, symbol Mechanical:MountingHole
Changed lines of the file:
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@@
+    )
+  )
+  (symbol (lib_id "Mechanical:MountingHole") (at 158.75 153.67 0) (unit 1)
+    (in_bom yes) (on_board yes) (dnp no) (fields_autoplaced)
+    (property "Reference" "H1" (at 161.29 153.0755 0)
+      (effects (font (size 1.27 1.27)) (justify left))
+    )
+    (property "Value" "MountingHole" (at 161.29 154.8377 0)
+      (effects (font (size 1.27 1.27)) (justify left))
+    )
+    (property "Footprint" "MountingHole:MountingHole_3.7mm_Pad_Via" (at 158.75 153.67 0)
+      (effects (font (size 1.27 1.27)) hide)
+    )
+    (property "Datasheet" "~" (at 158.75 153.67 0)
+      (effects (font (size 1.27 1.27)) hide)
+    )
+    (instances
+      (project "SSR8A"
+        (path "/6b7dd4b9-634f-41b4-b846-9b2e2d6d43c6"
+          (reference "H1") (unit 1) (value "MountingHole") (footprint "MountingHole:MountingHole_3.7mm_Pad_Via")
+        )
+      )
     )
   )

Commit message: WIP
Parts:
- added C14: 1u, Capacitor_SMD:C_0805_2012Metric_Pad1.18x1.45mm_HandSolder, symbol Device:C
- added R18: 10k, Resistor_SMD:R_0805_2012Metric_Pad1.20x1.40mm_HandSolder, symbol Device:R
- C2: renamed from C1; value C -> 10u
- C3: renamed from C2; value C -> 47u
- C4: renamed from C3; value C -> 47u
- J2: symbol Connector:Conn_01x03_Female -> Connector:Conn_01x03_Pin
- U3: renamed from U1; symbol Regulator_Linear:LM1117-3.3 -> Regulator_Linear:AMS1117-3.3
- renumbered R3 to R1, R1 to R2, R2 to R3, U2 to U1, U3 to U2
Connections:
- net +3V3: now also R18.1; no longer U2.2 (EN/CHIP_PU)
- net GND: now also C14.2
- new net: C14.1, R18.2, U2.2 (EN/CHIP_PU)

Commit message: WIP
Parts:
- U2: footprint Espressif:ESP32-C3-WROOM-02 -> Drake:ESP32-C3-WROOM-02 Handsolder
Changed lines of the file:
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@@
       (effects (font (size 1.27 1.27)))
     )
-    (property "Footprint" "Espressif:ESP32-C3-WROOM-02" (at 123.19 133.35 0)
+    (property "Footprint" "Drake:ESP32-C3-WROOM-02 Handsolder" (at 123.19 133.35 0)
       (effects (font (size 1.27 1.27)) hide)
     )
